Commit message: some changes for the simu

File: nexus_4wd_mecanum_description/urdf/nexus_4wd_mecanum.xacro (robot description, xacro)
@@ -345,3 +345,15 @@
     <xacro:zed_camera base_name="base_link" pos_x="-0.15" pos_y="0.0" pos_z="0.2" rotate_camera="1.0" camera_numb="4"/>
   </xacro:if>
+  <gazebo>
+      <plugin name="p3d_base_controller" filename="libgazebo_ros_p3d.so">
+            <alwaysOn>true</alwaysOn>
+            <updateRate>100.0</updateRate>
+            <bodyName>base_footprint</bodyName>
+            <topicName>ground_truth/pose</topicName>
+            <gaussianNoise>0.0</gaussianNoise>
+            <frameName>world</frameName>
+            <xyzOffsets>0 0 0</xyzOffsets>
+            <rpyOffsets>0 0 0</rpyOffsets>
+      </plugin>
+  </gazebo>
 </robot>

File: nexus_4wd_mecanum_description/urdf/zed_camera.urdf.xacro (robot description, xacro)
@@ -132,16 +132,16 @@
         </sensor>
     </gazebo>
-    <gazebo>
+    <!-- <gazebo>
       <plugin name="p3d_base_controller" filename="libgazebo_ros_p3d.so">
             <alwaysOn>true</alwaysOn>
-            <updateRate>50.0</updateRate>
-            <bodyName>left_camera_optical_frame_${numb}</bodyName>
+            <updateRate>100.0</updateRate>
+            <bodyName>base_footprint</bodyName>
             <topicName>ground_truth/left_camera_optical_frame_${numb}</topicName>
-            <gaussianNoise>0.001</gaussianNoise>
+            <gaussianNoise>0.0</gaussianNoise>
             <frameName>world</frameName>
             <xyzOffsets>0 0 0</xyzOffsets>
             <rpyOffsets>0 0 0</rpyOffsets>
       </plugin>
-  </gazebo>
-    </xacro:macro>
+  </gazebo> -->
+</xacro:macro>
 </robot>

Commit message: some changes

File: nexus_4wd_mecanum_description/urdf/nexus_4wd_mecanum.xacro (robot description, xacro)
@@ -150,5 +150,5 @@
     </inertial>
   </link>
-  <joint name="upper_left_wheel_joint" type="continuous">
+  <joint name="upper_left_wheel_joint" type="fixed">
     <origin xyz="0 0.042 0" rpy="0 0 0" />
     <parent link="upper_left_wheel_shaft"/>
@@ -180,5 +180,5 @@
     </inertial>
   </link>
-  <joint name="lower_left_wheel_joint" type="continuous">
+  <joint name="lower_left_wheel_joint" type="fixed">
     <origin xyz="0 0.042 0" rpy="0 0 0" />
     <parent link="lower_left_wheel_shaft"/>
@@ -210,5 +210,5 @@
     </inertial>
   </link>
-  <joint name="upper_right_wheel_joint" type="continuous">
+  <joint name="upper_right_wheel_joint" type="fixed">
     <origin xyz="0 0.042 0" rpy="0 0 0" />
     <parent link="upper_right_wheel_shaft"/>
@@ -240,5 +240,5 @@
     </inertial>
   </link>
-  <joint name="lower_right_wheel_joint" type="continuous">
+  <joint name="lower_right_wheel_joint" type="fixed">
     <origin xyz="0 0.042 0" rpy="0 0 0" />
     <parent link="lower_right_wheel_shaft"/>
@@ -270,5 +270,5 @@
     </inertial>
   </link>
-  <joint name="left_sensor_joint" type="fixed">
+  <!-- <joint name="left_sensor_joint" type="fixed">
     <origin xyz="0 0.108 0.010" rpy="0 0 ${PI/2}" />
     <parent link="base_link"/>
@@ -325,18 +325,20 @@
       <material name="black" />
     </visual>
-  </link>
-  <!-- Include controller plugin for Gazebo -->
+  </link> -->
   <xacro:include filename="$(find nexus_4wd_mecanum_description)/urdf/nexus_4wd_mecanum.gazebo" />
   <xacro:include filename="$(find nexus_4wd_mecanum_description)/urdf/zed_camera.urdf.xacro"/>
-  <!-- Include URM04 ultrasonic range finders -->
+  <!-- Include controller plugin for Gazebo -->
+  <!-- <xacro:include filename="$(find nexus_4wd_mecanum_description)/urdf/nexus_4wd_mecanum.gazebo" />
+  <xacro:include filename="$(find nexus_4wd_mecanum_description)/urdf/zed_camera.urdf.xacro"/>
+  Include URM04 ultrasonic range finders
   <xacro:include filename="$(find nexus_4wd_mecanum_description)/urdf/urm04_sensor.xacro"/>
-  <!-- front sensor -->
+  front sensor
   <xacro:urm04_sensor frame_name="front_sensor" ros_topic="front_sensor" update_rate="10" min_range="0.04" max_range="2.5" horizontal_field_of_view="1.04" vertical_field_of_view="0.04" ray_count="2" />
-  <!-- left sensor -->
+  left sensor
   <xacro:urm04_sensor frame_name="left_sensor" ros_topic="left_sensor" update_rate="10" min_range="0.04" max_range="2.5" horizontal_field_of_view="1.04" vertical_field_of_view="0.04" ray_count="2" />
-  <!-- right sensor -->
+  right sensor
   <xacro:urm04_sensor frame_name="right_sensor" ros_topic="right_sensor" update_rate="10" min_range="0.04" max_range="2.5" horizontal_field_of_view="1.04" vertical_field_of_view="0.04" ray_count="2" />
-  <!-- rear sensor -->
-  <xacro:urm04_sensor frame_name="rear_sensor" ros_topic="rear_sensor" update_rate="10" min_range="0.04" max_range="2.5" horizontal_field_of_view="1.04" vertical_field_of_view="0.04" ray_count="2" />
+  rear sensor
+  <xacro:urm04_sensor frame_name="rear_sensor" ros_topic="rear_sensor" update_rate="10" min_range="0.04" max_range="2.5" horizontal_field_of_view="1.04" vertical_field_of_view="0.04" ray_count="2" /> -->
   <xacro:zed_camera base_name="base_link" pos_x="0.15" pos_y="0.0" pos_z="0.2" rotate_camera="0.0" camera_numb="1"/>
   <xacro:if value="$(arg four_cameras)">

File: nexus_4wd_mecanum_description/urdf/zed_camera.urdf.xacro (robot description, xacro)
@@ -119,5 +119,5 @@
             <updateRate>0.0</updateRate>
             <cameraName>camera_${numb}</cameraName>
-            <imageTopicName>image_raw</imageTopicName>
+            <imageTopicName>image_rect</imageTopicName>
             <cameraInfoTopicName>camera_info</cameraInfoTopicName>
             <frameName>left_camera_optical_frame_${numb}</frameName>

Commit message: changes

File: nexus_4wd_mecanum_description/urdf/nexus_4wd_mecanum.xacro (robot description, xacro)
@@ -341,9 +341,9 @@
   rear sensor
   <xacro:urm04_sensor frame_name="rear_sensor" ros_topic="rear_sensor" update_rate="10" min_range="0.04" max_range="2.5" horizontal_field_of_view="1.04" vertical_field_of_view="0.04" ray_count="2" /> -->
-  <xacro:zed_camera base_name="base_link" pos_x="0.15" pos_y="0.0" pos_z="0.2" rotate_camera="0.0" camera_numb="1"/>
+  <xacro:zed_camera base_name="base_link" pos_x="0.15" pos_y="0.0" pos_z="0.2" rotate_camera="0.0" camera_numb="1" reshh = "480" resww = "752"/>
   <xacro:if value="$(arg four_cameras)">
-    <xacro:zed_camera base_name="base_link" pos_x="0.0" pos_y="-0.15" pos_z="0.2" rotate_camera="-0.5" camera_numb="2"/>
-    <xacro:zed_camera base_name="base_link" pos_x="0.0" pos_y="0.15" pos_z="0.2" rotate_camera="0.5" camera_numb="3"/>
-    <xacro:zed_camera base_name="base_link" pos_x="-0.15" pos_y="0.0" pos_z="0.2" rotate_camera="1.0" camera_numb="4"/>
+    <xacro:zed_camera base_name="base_link" pos_x="0.0" pos_y="-0.15" pos_z="0.2" rotate_camera="-0.5" camera_numb="2" reshh = "1080" resww = "1920"/>
+    <!-- <xacro:zed_camera base_name="base_link" pos_x="0.0" pos_y="0.15" pos_z="0.2" rotate_camera="0.5" camera_numb="3" reshh = "480" resww = "752"/> -->
+    <xacro:zed_camera base_name="base_link" pos_x="-0.15" pos_y="0.0" pos_z="0.2" rotate_camera="1.0" camera_numb="4" reshh = "480" resww = "752"/>
   </xacro:if>
   <gazebo>

File: nexus_4wd_mecanum_description/urdf/zed_camera.urdf.xacro (robot description, xacro)
@@ -1,5 +1,5 @@
 <?xml version="1.0"?>
 <robot xmlns:xacro="http://ros.org/wiki/xacro">
-    <xacro:macro name="zed_camera" params="base_name pos_x pos_y pos_z rotate_camera camera_numb" >
+    <xacro:macro name="zed_camera" params="base_name pos_x pos_y pos_z rotate_camera camera_numb reshh resww" >
     <!-- Arguments -->
     <xacro:arg name="camera_name"   default="zed2" />
@@ -17,4 +17,6 @@
     <xacro:property name="rotate"        value="${rotate_camera}" />
     <xacro:property name="numb"          value="${camera_numb}" />
+    <xacro:property name="resh"          value="${reshh}" />
+    <xacro:property name="resw"          value="${resww}" />
     <!-- Materials -->
     <material name="zed_mat_${numb}">
@@ -84,5 +86,5 @@
     <gazebo reference="left_camera_frame_${numb}">
         <sensor type="multicamera" name="stereo_camera">
-        <update_rate>10.0</update_rate>
+        <update_rate>15.0</update_rate>
         <camera name="left">
             <horizontal_fov>1.91986218</horizontal_fov>
@@ -90,6 +92,6 @@
             <diagonal_fov>2.0943951</diagonal_fov>
             <image>
-                <width>752</width>
-                <height>480</height>
+                <width>${resw}</width>
+                <height>${resh}</height>
                 <format>R8G8B8</format>
             </image>
@@ -105,6 +107,6 @@
             <diagonal_fov>2.0943951</diagonal_fov>
             <image>
-                <width>752</width>
-                <height>480</height>
+                <width>${resw}</width>
+                <height>${resh}</height>
                 <format>R8G8B8</format>
             </image>
